File: kicad_pcb_model/final/esp32-wavplayer-final.kicad_sch (KiCad schematic)
At the start: 92 parts, among them J1 BIN+, J2 BIN-, SW1 RST, SW2 BOOT, U3 PCM5102A

Commit message: Powerstage redesign
Parts:
- added BD1, BD2: D, Diode_SMD:D_0603_1608Metric_Pad1.05x0.95mm_HandSolder, symbol Device:D
- added BR3: 4.7k, Resistor_SMD:R_0603_1608Metric_Pad0.98x0.95mm_HandSolder, symbol Device:R
- added BR4: 6.8k, Resistor_SMD:R_0603_1608Metric_Pad0.98x0.95mm_HandSolder, symbol Device:R
- added BR5: 15k, Resistor_SMD:R_0603_1608Metric_Pad0.98x0.95mm_HandSolder, symbol Device:R
- added SW3: RIGHT, Button_Switch_SMD:SW_SPST_TS-1088-xR020, symbol Switch:SW_Push
- added SW4: LEFT, Button_Switch_SMD:SW_SPST_TS-1088-xR020, symbol Switch:SW_Push
- added SW5: DOWN, Button_Switch_SMD:SW_SPST_TS-1088-xR020, symbol Switch:SW_Push
- SW2: value BOOT -> BOOT/UP
Connections:
- net GPIO18/USB_D- is gone; now on net GPIO19/USB_D-: CPU1.25 (GPIO18/USB_D-)
- net GPIO19/USB_D+ is gone; now on net GPIO18/USB_D+: CPU1.26 (GPIO19/USB_D+)
- net +3V3: now also BR3.1, BR4.1, BR5.1; no longer BTM1.5 (BAT), J1.1 (Pin_1), PC4.1, PC5.1, PR7.2
- net Earth: now also SW3.1, SW4.1, SW5.1
- net GPIO9: now also BD2.1 (K); no longer BR2.2, SW2.2
- net VSYS: no longer PC1.1, PDVR1.1 (V_{IN}), PDVR1.3 (CE)
- net GPIO10: now reaches CPU1.16 (GPIO10)
- net UARTRX: now reaches CPU1.27 (U0RXD/GPIO20)
- net UARTTX: now reaches CPU1.28 (U0TXD/GPIO21)
- net ANALOG_INPUT: now reaches CPU1.4 (XTAL_32K_P/ADC1_CH0)
- net ANALOG_INPUT: now also BD1.1 (K), BR3.2, BR4.2, BR5.2, SW3.2, SW4.2, SW5.2
- new net: PC1.1, PC5.1, PDVR1.1 (V_{IN}), PDVR1.3 (CE)
- new net: BD1.2 (A), BD2.2 (A), BR2.2, SW2.2
- new net: BTM1.5 (BAT), J1.1 (Pin_1), PC4.1, PR7.2
- no-connect marks 5 -> 12
Other:
- moved on the sheet: BC1, BR1, BR2, D3, D4, LR1, LR2, SW1, SW2

Commit message: Fixing shiz
Parts:
- removed DC2: C, Capacitor_SMD:C_0603_1608Metric_Pad1.08x0.95mm_HandSolder, symbol Device:C
- removed OC1: 15pF, Capacitor_SMD:C_0603_1608Metric_Pad1.08x0.95mm_HandSolder, symbol Device:C
- added BB1: TPS63900, Package_SON:WSON-10-1EP_2.5x2.5mm_P0.5mm_EP1.2x2mm_ThermalVias, symbol Regulator_Switching:TPS63900
- added DB4: DebugPinVbat, symbol Connector:Conn_01x01_Pin
- added OC3: 15pF, Capacitor_SMD:C_0603_1608Metric_Pad1.08x0.95mm_HandSolder, symbol Device:C
- AC12, AC13: value 2.2uF -> 2.2nF
- CPU1: value ESP32-C3 -> ESP32-C3-H*
- DC3, DC4, DC5, DC6: value C -> 1uF
Connections:
- net RES# is gone; now on net GPIO9: DS1.14 (~{RES})
- net Earth: now also CYOC1.4 (Vdd), OC3.2; no longer CYOC1.1 (EN), DS1.17 (E/~{RD})
- net VDD: now also DS1.17 (E/~{RD})
- net XTAL_N: now also CYOC1.1 (EN), OC3.1; no longer CYOC1.3 (OUT), OC2.1
- net XTAL_P: now also CYOC1.3 (OUT), OC2.1; no longer CYOC1.4 (Vdd)
- net at AC10.1, AC9.1, AR3.1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: now also U3.17 (XSMT)
- net at AC2.1, AC3.1, AC4.1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: no longer U3.17 (XSMT)
- net at DS1.6 (VBAT): now also DB4.1 (Pin_1)
- new net: BB1.11 (GND), BB1.8 (GND)
Other:
- note added: "Regulate ldo output to 3.5v"
- moved on the sheet: DC1, OC2

Commit message: updated wisevision configuration
Parts:
- removed BB1: TPS63900, Package_SON:WSON-10-1EP_2.5x2.5mm_P0.5mm_EP1.2x2mm_ThermalVias, symbol Regulator_Switching:TPS63900
- added BB1: TPS63030DSK, Package_SON:WSON-10-1EP_2.5x2.5mm_P0.5mm_EP1.2x2mm, symbol Regulator_Switching:TPS63030DSK
- added BCC1: 0.1uF, Capacitor_SMD:C_0603_1608Metric_Pad1.08x0.95mm_HandSolder, symbol Device:C
- added BCC2, BCC3: 10uF, Capacitor_SMD:C_0603_1608Metric_Pad1.08x0.95mm_HandSolder, symbol Device:C
- added BCL1: 2.2uH, symbol Device:L
- added BCR1: 200k, Resistor_SMD:R_0603_1608Metric_Pad0.98x0.95mm_HandSolder, symbol Device:R
- added BCR2: 1.2M, Resistor_SMD:R_0603_1608Metric_Pad0.98x0.95mm_HandSolder, symbol Device:R
- added DQ1: FDN338P, Package_TO_SOT_SMD:SOT-23, symbol Transistor_FET:FDN340P
- added DQ2: FDN335N, Package_TO_SOT_SMD:SOT-23, symbol Transistor_FET:FDN340P
- added DR4, DR5: 47k, Resistor_SMD:R_0603_1608Metric_Pad0.98x0.95mm_HandSolder, symbol Device:R
- DC1: value C -> 2.2uF
- DC7: value C -> 4.7uF
- DR1, DR2: value R -> 4.7k
- DR3: value R -> 620k
Connections:
- net +3V3: now also DC3.1, DC4.2, DR1.1, DR2.1, DS1.11 (BS1), DS1.9 (VDD), BB1.5 (VIN), BB1.6 (EN), BB1.7 (PS/SYNC), BCC2.2, DR4.2
- net Earth: now also DS1.17 (E/~{RD}), BB1.11 (PGND), BB1.3 (PGND), BB1.9 (GND), BCC1.1, BCC2.1, BCC3.1, BCR2.2, DQ2.2 (S), DR5.2
- net VBAT: now reaches DB4.1 (Pin_1), DS1.6 (VBAT)
- net VBAT: now also DQ1.2 (S)
- removed net VDD: DC3.1, DC4.2, DR1.1, DR2.1, DS1.11 (BS1), DS1.17 (E/~{RD}), DS1.9 (VDD)
- new net: DQ1.1 (G), DQ2.3 (D), DR4.1
- new net: BB1.4 (L1), BCL1.1
- new net: BB1.2 (L2), BCL1.2
- new net: BB1.8 (VINA), BCC1.2
- new net: BB1.10 (FB), BCR1.2, BCR2.1
- new net BATT: BB1.1 (VOUT), BCC3.2, BCR1.1, DQ1.3 (D)
- new net GPIO: DQ2.1 (G), DR5.1
Other:
- note removed: "Regulate ldo output to 3.5v"
- moved on the sheet: A1, AC1, AC10, AC11, AC12, AC13, AC14, AC2, AC3, AC4, AC5, AC6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

Commit message: updating model
Parts:
- BCL1: footprint (none) -> Inductor_SMD:L_0201_0603Metric_Pad0.64x0.40mm_HandSolder
- DB4: footprint (none) -> Connector_PinHeader_2.54mm:PinHeader_1x01_P2.54mm_Vertical
Changed lines of the file:
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@@
 			)
 		)
-		(property "Footprint" ""
+		(property "Footprint" "Connector_PinHeader_2.54mm:PinHeader_1x01_P2.54mm_Vertical"
 			(at 254 78.74 0)
 			(hide yes)
@@
 			)
 		)
-		(property "Footprint" ""
+		(property "Footprint" "Inductor_SMD:L_0201_0603Metric_Pad0.64x0.40mm_HandSolder"
 			(at 207.01 72.39 0)
 			(hide yes)

Commit message: fixed battery connection
Parts:
- removed PC5: 10uF, Capacitor_SMD:C_0603_1608Metric_Pad1.08x0.95mm_HandSolder, symbol Device:C
- added J3: DBG3v3, Connector_PinHeader_2.54mm:PinHeader_1x01_P2.54mm_Vertical, symbol Connector:Conn_01x01_Pin
Connections:
- net +3V3: now also J3.1 (Pin_1)
- net at PC1.1, PDVR1.1 (V_{IN}), PDVR1.3 (CE): now also BTM1.5 (BAT), J1.1 (Pin_1), PC4.1, PR7.2
- no-connect marks 12 -> 13
Changed lines of the file:
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@@
 	)
 	(junction
+		(at 146.05 21.59)
+		(diameter 0)
+		(color 0 0 0 0)
+	)
+	(junction
 		(at 22.86 76.2)
 		(diameter 0)
@@
 	)
 	(junction
-		(at 189.23 21.59)
-		(diameter 0)
-		(color 0 0 0 0)
-	)
-	(junction
 		(at 184.15 97.79)
 		(diameter 0)
@@
 	)
 	(no_connect
+		(at 114.3 48.26)
+	)
+	(no_connect
 		(at 191.77 43.18)
 	)
@@
 	(wire
 		(pts
-			(xy 189.23 20.32) (xy 189.23 21.59)
+			(xy 189.23 20.32) (xy 189.23 33.02)
 		)
 		(stroke
@@
 	(wire
 		(pts
-			(xy 182.88 21.59) (xy 189.23 21.59)
-		)
-		(stroke
-			(width 0)
-			(type default)
-		)
-	)
-	(wire
-		(pts
 			(xy 257.81 118.11) (xy 246.38 118.11)
 		)
@@
 	(wire
 		(pts
+			(xy 146.05 21.59) (xy 146.05 13.97)
+		)
+		(stroke
+			(width 0)
+			(type default)
+		)
+	)
+	(wire
+		(pts
 			(xy 116.84 49.53) (xy 116.84 48.26)
 		)
@@
 	(wire
 		(pts
-			(xy 175.26 21.59) (xy 170.18 21.59)
+			(xy 30.48 102.87) (xy 46.99 102.87)
 		)
 		(stroke
@@
 	(wire
 		(pts
-			(xy 30.48 102.87) (xy 46.99 102.87)
+			(xy 280.67 71.12) (xy 273.05 71.12)
 		)
 		(stroke
@@
 	(wire
 		(pts
-			(xy 280.67 71.12) (xy 273.05 71.12)
+			(xy 13.97 168.91) (xy 13.97 170.18)
 		)
 		(stroke
@@
 	(wire
 		(pts
-			(xy 13.97 168.91) (xy 13.97 170.18)
+			(xy 134.62 142.24) (xy 134.62 134.62)
 		)
 		(stroke
@@
 	(wire
 		(pts
-			(xy 134.62 142.24) (xy 134.62 134.62)
+			(xy 222.25 88.9) (xy 223.52 88.9)
 		)
 		(stroke
@@
 	(wire
 		(pts
-			(xy 222.25 88.9) (xy 223.52 88.9)
+			(xy 146.05 21.59) (xy 149.86 21.59)
 		)
 		(stroke
@@
 	(wire
 		(pts
+			(xy 76.2 20.32) (xy 73.66 20.32)
+		)
+		(stroke
+			(width 0)
+			(type default)
+		)
+	)
+	(wire
+		(pts
 			(xy 195.58 59.69) (xy 207.01 59.69)
 		)
@@
 	(wire
 		(pts
+			(xy 146.05 13.97) (xy 45.72 13.97)
+		)
+		(stroke
+			(width 0)
+			(type default)
+		)
+	)
+	(wire
+		(pts
 			(xy 220.98 45.72) (xy 240.03 45.72)
 		)
@@
 	(wire
 		(pts
-			(xy 170.18 13.97) (xy 170.18 21.59)
-		)
-		(stroke
-			(width 0)
-			(type default)
-		)
-	)
-	(wire
-		(pts
 			(xy 226.06 123.19) (xy 257.81 123.19)
 		)
@@
 	(wire
 		(pts
-			(xy 189.23 21.59) (xy 189.23 33.02)
-		)
-		(stroke
-			(width 0)
-			(type default)
-		)
-	)
-	(wire
-		(pts
 			(xy 257.81 85.09) (xy 245.11 85.09)
 		)
@@
 	(wire
 		(pts
-			(xy 170.18 13.97) (xy 45.72 13.97)
-		)
-		(stroke
-			(width 0)
-			(type default)
-		)
-	)
-	(wire
-		(pts
 			(xy 149.86 123.19) (xy 158.75 123.19)
 		)
@@
 	(wire
 		(pts
-			(xy 127 21.59) (xy 149.86 21.59)
+			(xy 127 21.59) (xy 146.05 21.59)
 		)
 		(stroke
@@
 	)
 	(symbol
+		(lib_id "Connector:Conn_01x01_Pin")
+		(at 81.28 20.32 180)
+		(unit 1)
+		(body_style 1)
+		(exclude_from_sim no)
+		(in_bom yes)
+		(on_board yes)
+		(in_pos_files yes)
+		(dnp no)
+		(fields_autoplaced yes)
+		(property "Reference" "J3"
+			(at 80.645 15.24 0)
+			(show_name no)
+			(do_not_autoplace no)
+			(effects
+				(font
+					(size 1.27 1.27)
+				)
+			)
+		)
+		(property "Value" "DBG3v3"
+			(at 80.645 17.78 0)
+			(show_name no)
+			(do_not_autoplace no)
+			(effects
+				(font
+					(size 1.27 1.27)
+				)
+			)
+		)
+		(property "Footprint" "Connector_PinHeader_2.54mm:PinHeader_1x01_P2.54mm_Vertical"
+			(at 81.28 20.32 0)
+			(hide yes)
+			(show_name no)
+			(do_not_autoplace no)
+			(effects
+				(font
+					(size 1.27 1.27)
+				)
+			)
+		)
+		(property "Datasheet" ""
+			(at 81.28 20.32 0)
+			(hide yes)
+			(show_name no)
+			(do_not_autoplace no)
+			(effects
+				(font
+					(size 1.27 1.27)
+				)
+			)
+		)
+		(property "Description" "Generic connector, single row, 01x01, script generated"
+			(at 81.28 20.32 0)
+			(hide yes)
+			(show_name no)
+			(do_not_autoplace no)
+			(effects
+				(font
+					(size 1.27 1.27)
+				)
+			)
+		)
+		(pin "1"
+		)
+		(instances
+			(project "esp32-wavplayer-final"
+				(path "/e8fbce24-19e4-4fd2-98dc-690d4768f544"
+					(reference "J3")
+					(unit 1)
+				)
+			)
+		)
+	)
+	(symbol
 		(lib_id "Device:C")
 		(at 24.13 120.65 0)
@@
 					(unit 1)
 				)
-			)
-		)
-	)
-	(symbol
-		(lib_id "Device:C")
-		(at 179.07 21.59 90)
-		(unit 1)
-		(body_style 1)
-		(exclude_from_sim no)
-		(in_bom yes)
-		(on_board yes)
-		(in_pos_files yes)
-		(dnp no)
-		(property "Reference" "PC5"
-			(at 177.546 20.574 90)
-			(show_name no)
-			(do_not_autoplace no)
-			(effects
-				(font
-					(size 1.27 1.27)
-				)
-				(justify left)
-			)
-		)
-		(property "Value" "10uF"
-			(at 184.658 20.574 90)
-			(show_name no)
-			(do_not_autoplace no)
-			(effects
-				(font
-					(size 1.27 1.27)
-				)
-				(justify left)
-			)
-		)
-		(property "Footprint" "Capacitor_SMD:C_0603_1608Metric_Pad1.08x0.95mm_HandSolder"
-			(at 182.88 20.6248 0)
-			(hide yes)
-			(show_name no)
-			(do_not_autoplace no)
-			(effects
-				(font
-					(size 1.27 1.27)
-				)
-			)
-		)
-		(property "Datasheet" ""
-			(at 179.07 21.59 0)
-			(hide yes)
-			(show_name no)
-			(do_not_autoplace no)
-			(effects
-				(font
-					(size 1.27 1.27)
-				)
-			)
-		)
-		(property "Description" "Unpolarized capacitor"
-			(at 179.07 21.59 0)
-			(hide yes)
-			(show_name no)
-			(do_not_autoplace no)
-			(effects
-				(font
-					(size 1.27 1.27)
-				)
-			)
-		)
-		(pin "2"
-		)
-		(pin "1"
-		)
-		(instances
-			(project "esp32-wavplayer-final"
-				(path "/e8fbce24-19e4-4fd2-98dc-690d4768f544"
-					(reference "PC5")
-					(unit 1)
-				)
